File: oal-sapphire-psu.sch (KiCad schematic (older format))
At the start: 35 parts, among them P1 IEC, P2 LINE, P3 NEUTRAL, P4 PRIMARY_4, P5 PRIMARY_5, P6 SWITCHED_LINE, P7 OUTPUT, T1 TALEMA-25VA/12V, X1 MOUNTING_HOLE, X2 MOUNTING_HOLE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

Commit message: updated layout
Parts:
- P7: footprint Terminal_Blocks:TerminalBlock_Pheonix_PT-3.5mm_6pol -> ose-audio-labs:TerminalBlock_Pheonix_PT-3.5mm_6pol-Vertical
- R1, R2: value 820R -> 680R
Changed lines of the file:
@@
 LIBS:valves
 LIBS:ose-audio-labs
-LIBS:switch_dpdt
-LIBS:oal-sapphire-rectifier-cache
+LIBS:oal-sapphire-psu-cache
 EELAYER 25 0
 EELAYER END
@@
 P 7150 5175
 F 0 "R1" V 7230 5175 50  0000 C CNN
-F 1 "820R" V 7150 5175 50  0000 C CNN
+F 1 "680R" V 7150 5175 50  0000 C CNN
 F 2 "Resistors_SMD:R_0805" V 7080 5175 50  0001 C CNN
 F 3 "" H 7150 5175 50  0000 C CNN
@@
 P 6750 5575
 F 0 "R2" V 6830 5575 50  0000 C CNN
-F 1 "820R" V 6750 5575 50  0000 C CNN
+F 1 "680R" V 6750 5575 50  0000 C CNN
 F 2 "Resistors_SMD:R_0805" V 6680 5575 50  0001 C CNN
 F 3 "" H 6750 5575 50  0000 C CNN
@@
 F 0 "P7" H 7619 2100 50  0000 C CNN
 F 1 "OUTPUT" H 7619 2191 50  0000 C CNN
-F 2 "Terminal_Blocks:TerminalBlock_Pheonix_PT-3.5mm_6pol" H 7700 2575 50  0001 C CNN
+F 2 "ose-audio-labs:TerminalBlock_Pheonix_PT-3.5mm_6pol-Vertical" H 7700 2575 50  0001 C CNN
 F 3 "" H 7700 2575 50  0000 C CNN
 	1    7700 2575
